File: Hardware/vesc4-raw/after-remap/temp.kicad_sch (KiCad schematic)
At the start: 3 parts

Commit message: export footprint & ngapus warning unmatched
Parts:
- C41: symbol after-remap-rescue:C-RESCUE-BLDC_4 -> vesc4-legacy:C-RESCUE-BLDC_4_2
- R1: symbol after-remap-rescue:R-RESCUE-BLDC_4 -> vesc4-legacy:R-RESCUE-BLDC_4_3
- R2: symbol after-remap-rescue:R-RESCUE-BLDC_4 -> vesc4-legacy:R-RESCUE-BLDC_4_4
Changed lines of the file:
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@@
 	(symbol
 		(lib_name "R-RESCUE-BLDC_4_3")
-		(lib_id "after-remap-rescue:R-RESCUE-BLDC_4")
+		(lib_id "vesc4-legacy:R-RESCUE-BLDC_4_3")
 		(at 111.76 86.36 0)
 		(unit 1)
@@
 	(symbol
 		(lib_name "R-RESCUE-BLDC_4_4")
-		(lib_id "after-remap-rescue:R-RESCUE-BLDC_4")
+		(lib_id "vesc4-legacy:R-RESCUE-BLDC_4_4")
 		(at 111.76 104.14 0)
 		(unit 1)
@@
 	(symbol
 		(lib_name "C-RESCUE-BLDC_4_2")
-		(lib_id "after-remap-rescue:C-RESCUE-BLDC_4")
+		(lib_id "vesc4-legacy:C-RESCUE-BLDC_4_2")
 		(at 105.41 104.14 0)
 		(unit 1)
@@
 	(symbol
 		(lib_name "VCC_2")
-		(lib_id "after-remap-rescue:VCC")
+		(lib_id "vesc4-legacy:VCC_2")
 		(at 111.76 77.47 0)
 		(unit 1)
@@
 	(symbol
 		(lib_name "GND-RESCUE-BLDC_4_2")
-		(lib_id "after-remap-rescue:GND-RESCUE-BLDC_4")
+		(lib_id "vesc4-legacy:GND-RESCUE-BLDC_4_2")
 		(at 111.76 116.84 0)
 		(unit 1)
