File: Hardware/vesc4-raw/after-remap/temp.kicad_sch (KiCad schematic)
At the start: 3 parts

Commit message: chekcpoint 18 mei
Parts:
- C41: footprint CRF1:SMD-0603_c -> easypretty:C0603; JLC_3DModel (none) -> ac9b32e974bc448eab36b1293f859dcb; JLC_3D_Size (none) -> 1.6 0.8; LCSC (none) -> C23630; LCSC Part (none) -> C1631
- R1, R2: footprint Library:R0603 -> easypretty:R0603; LCSC (none) -> C25804; LCSC Part (none) -> C23164
Changed lines of the file:
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@@
 			)
 		)
-		(property "Footprint" "Library:R0603"
+		(property "Footprint" "easypretty:R0603"
 			(at 109.982 86.36 90)
 			(effects
@@
 		)
 		(property "JLC_3D_Size" "0.81 1.62"
+			(at 111.76 86.36 0)
+			(effects
+				(font
+					(size 1.27 1.27)
+				)
+				(hide yes)
+			)
+		)
+		(property "LCSC" "C25804"
+			(at 111.76 86.36 0)
+			(effects
+				(font
+					(size 1.27 1.27)
+				)
+				(hide yes)
+			)
+		)
+		(property "LCSC Part" "C23164"
 			(at 111.76 86.36 0)
 			(effects
@@
 			)
 		)
-		(property "Footprint" "Library:R0603"
+		(property "Footprint" "easypretty:R0603"
 			(at 109.982 104.14 90)
 			(effects
@@
 		)
 		(property "JLC_3D_Size" "0.81 1.62"
+			(at 111.76 104.14 0)
+			(effects
+				(font
+					(size 1.27 1.27)
+				)
+				(hide yes)
+			)
+		)
+		(property "LCSC" "C25804"
+			(at 111.76 104.14 0)
+			(effects
+				(font
+					(size 1.27 1.27)
+				)
+				(hide yes)
+			)
+		)
+		(property "LCSC Part" "C23164"
 			(at 111.76 104.14 0)
 			(effects
@@
 			)
 		)
-		(property "Footprint" "CRF1:SMD-0603_c"
+		(property "Footprint" "easypretty:C0603"
 			(at 106.3752 107.95 0)
 			(effects
@@
 			)
 		)
+		(property "JLC_3DModel" "ac9b32e974bc448eab36b1293f859dcb"
+			(at 105.41 104.14 0)
+			(effects
+				(font
+					(size 1.27 1.27)
+				)
+				(hide yes)
+			)
+		)
+		(property "JLC_3D_Size" "1.6 0.8"
+			(at 105.41 104.14 0)
+			(effects
+				(font
+					(size 1.27 1.27)
+				)
+				(hide yes)
+			)
+		)
+		(property "LCSC" "C23630"
+			(at 105.41 104.14 0)
+			(effects
+				(font
+					(size 1.27 1.27)
+				)
+				(hide yes)
+			)
+		)
+		(property "LCSC Part" "C1631"
+			(at 105.41 104.14 0)
+			(effects
+				(font
+					(size 1.27 1.27)
+				)
+				(hide yes)
+			)
+		)
