File: Hardware/vesc4-raw/after-remap/after-remap.kicad_sch (KiCad schematic)
At the start: 26 parts, among them K1 SERVO, P1 HALL/Encoder, P101 CANBUS, P3 PWR_COMM, P4 IN+, P5 IN-, P6 MOTOR1, P7 MOTOR2, P9 MOTOR3, U4 MICROQTJ

Commit message: all done
Parts:
- P1: footprint CRF1:MICRO_JST_6 -> Library:CONN-TH_B6B-PH-K-S
- P101: footprint JST conn:b4b-ph-kl -> Library:CONN-TH_B4B-PH-K-S
- P3: footprint CRF1:b7b-ph-kl -> Library:CONN-TH_B7B-PH-K-S-LF-SN
Changed lines of the file:
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@@
 			)
 		)
-		(property "Footprint" "CRF1:MICRO_JST_6"
+		(property "Footprint" "Library:CONN-TH_B6B-PH-K-S"
 			(at 27.94 118.11 0)
 			(effects
@@
 			)
 		)
-		(property "Footprint" "JST conn:b4b-ph-kl"
+		(property "Footprint" "Library:CONN-TH_B4B-PH-K-S"
 			(at 27.94 100.33 0)
 			(effects
@@
 			)
 		)
-		(property "Footprint" "CRF1:b7b-ph-kl"
+		(property "Footprint" "Library:CONN-TH_B7B-PH-K-S-LF-SN"
 			(at 31.75 140.97 0)
 			(effects

Commit message: chekcpoint 18 mei
Parts:
- added R6: 10k, easypretty:R0603, symbol vesc4-legacy:R-RESCUE-BLDC_4_13
- C2, C3: footprint Library:C0603 -> easypretty:C0603; LCSC (none) -> C14663; LCSC Part (none) -> C1631
- D1: footprint Library:LED0603-R-RD_WHITE -> easypretty:LED0603-R-RD_WHITE; LCSC (none) -> C2905797; LCSC Part (none) -> C2290
- D2: footprint Library:LED0603-R-RD_WHITE -> easypretty:LED0603-R-RD_WHITE; LCSC (none) -> C2904374; LCSC Part (none) -> C2290
- D3: footprint Library:LED0603-R-RD_WHITE -> easypretty:LED0603-R-RD_WHITE; LCSC (none) -> C2290; LCSC Part (none) -> C2290
- D6: JLC_3DModel_Q (none) -> cdc13862fe374d3bb7a14a8cac9d9007; JLC_3D_Size (none) -> 5.05 2.6; LCSC (none) -> C14238
- P1: footprint Library:CONN-TH_B6B-PH-K-S -> easypretty:CONN-TH_B6B-PH-K-S
- P101: footprint Library:CONN-TH_B4B-PH-K-S -> easypretty:CONN-TH_B4B-PH-K-S
- P3: footprint Library:CONN-TH_B7B-PH-K-S-LF-SN -> easypretty:CONN-TH_B7B-PH-K-S-LF-SN
- R103, R104: footprint Library:R0603 -> easypretty:R0603; LCSC (none) -> C23345; LCSC Part (none) -> C23164
- R22, R4, R5: footprint Library:R0603 -> easypretty:R0603; LCSC (none) -> C4190; LCSC Part (none) -> C23164
- R3: footprint Library:R0603 -> easypretty:R0603; LCSC (none) -> C23153; LCSC Part (none) -> C23164
- R37, R38: footprint Library:R0603 -> easypretty:R0603; LCSC (none) -> C22775; LCSC Part (none) -> C23164
- R53, R54: footprint Library:C2076510 -> easypretty:R2726; JLC_3DModel (none) -> 76bc509a5511445c8d320e01eb58c99c; JLC_3D_Size (none) -> 6.9 6.6; LCSC (none) -> C2076510; LCSC Part (none) -> C2076510
- U4: footprint Library:MICRO-USB-SMD_MICROQTJ-5P -> easypretty:MICRO-USB-SMD_MICROQTJ-5P; LCSC (none) -> C404968; LCSC Part (none) -> C404968
Connections:
- net MISO_RX_SCL: now also R6.2
- net VCC: now also R6.1

Commit message: cp1
Parts:
- D1: LCSC C2905797 -> C125098
- D2: LCSC C2904374 -> C125099
- D6: footprint EasyEDA_Lib:SMA_L4.2-W2.6-LS5.1-RD -> easypretty:SOD-123_L2.8-W1.8-LS3.7-RD; LCSC C14238 -> C98663; LCSC Part (none) -> C98663
- R53, R54: LCSC C2076510 -> C500635
- R6: LCSC C25819 -> C25804
Changed lines of the file:
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@@
 			)
 		)
-		(property "LCSC" "C2904374"
+		(property "LCSC" "C125099"
 			(at 149.86 173.99 0)
 			(effects
@@
 			)
 		)
-		(property "LCSC" "C2905797"
+		(property "LCSC" "C125098"
 			(at 157.48 173.99 0)
 			(effects
@@
 			)
 		)
-		(property "LCSC" "C2076510"
+		(property "LCSC" "C500635"
 			(at 213.36 123.19 0)
 			(effects
@@
 			)
 		)
-		(property "LCSC" "C25819"
+		(property "LCSC" "C25804"
 			(at 44.45 156.21 0)
 			(effects
@@
 			)
 		)
-		(property "LCSC" "C2076510"
+		(property "LCSC" "C500635"
 			(at 203.2 110.49 0)
 			(effects
@@
 			)
 		)
-		(property "Footprint" "EasyEDA_Lib:SMA_L4.2-W2.6-LS5.1-RD"
+		(property "Footprint" "easypretty:SOD-123_L2.8-W1.8-LS3.7-RD"
 			(at 59.69 74.93 0)
 			(effects
@@
 			)
 		)
-		(property "Datasheet" "https://atta.szlcsc.com/upload/public/pdf/source/20190416/C379823_9D66F8781E151C8A4940396CFA0EFE63.pdf"
+		(property "Datasheet" ""
 			(at 59.69 74.93 0)
 			(effects
@@
 			)
 		)
-		(property "Description" "Forward Voltage (Vf@If):850mV@1A Reverse Voltage (Vr):100V Average Rectified Current (Io):1A"
+		(property "Description" ""
 			(at 59.69 74.93 0)
 			(effects
@@
 			)
 		)
-		(property "LCSC" "C14238"
+		(property "LCSC" "C98663"
 			(at 59.69 74.93 0)
 			(effects
+				(font
+					(size 1.27 1.27)
+				)
+				(hide yes)
+			)
+		)
+		(property "LCSC Part" "C98663"
+			(at 59.69 74.93 0)
+			(effects

Commit message: cp23mei
Parts:
- added H1, H2, H3, H4: MountingHole, MountingHole:MountingHole_3.2mm_M3_DIN965_Pad, symbol Mechanical:MountingHole
- added H5: MountingHole_Pad, MountingHole:MountingHole_3.2mm_M3_DIN965_Pad, symbol Mechanical:MountingHole_Pad
Connections:
- net GND: now also R53.4, R54.3; no longer R53.3, R54.4
- net Mosfet driver/H1_LOW: no longer R53.4
- net Mosfet driver/H3_LOW: now also R53.3, R54.4; no longer R54.3
- net V_SUPPLY: now also H5.1

Commit message: cp29mei
Parts:
- added D7: LED, easypretty:LED0603-R-RD_WHITE, symbol vesc4-legacy:LED-RESCUE-BLDC_4_6
- added H6, H7, H8: MountingHole, MountingHole:MountingHole_3.2mm_M3_DIN965_Pad, symbol Mechanical:MountingHole_Pad
- added H9: MountingHole_Pad, MountingHole:MountingHole_3.2mm_M3_DIN965_Pad, symbol Mechanical:MountingHole_Pad
- added R14: 2k2, easypretty:R0603, symbol vesc4-legacy:R-RESCUE-BLDC_4_15
- P4, P5, P6, P7, P9: footprint CRF1:1PAD_4x5mm -> Library:PAD
Connections:
- net +5V: now also R14.2
- net GND: now also D7.2 (K), H9.1
- net Mosfet driver/H1_LOW: now also R54.4
- net Mosfet driver/H3_LOW: no longer R54.4
- net Power MOSFETS/PHASE_1: now also P6.1, H6.1; no longer P9.1
- net Power MOSFETS/PHASE_2: now also H7.1
- net Power MOSFETS/PHASE_3: now also P9.1, H8.1; no longer P6.1
- net MCU/USB_DM renamed USB-
- net MCU/USB_DP renamed USB+
- net Mosfet driver/SH1_A renamed SH1+
- net Mosfet driver/SH1_B renamed SH1-
- net Mosfet driver/SH2_A renamed SH2-
- net Mosfet driver/SH2_B renamed SH2+
- new net: D7.1 (A), R14.1
Other:
- moved on the sheet: P6, P7, P9

Commit message: 16-06-2026
Parts:
- added ADCbp1: PWR_COMM, Library:CONN-TH_B7B-PH-K-S-LF-SN, symbol vesc4-legacy:CONN_01X07_2
- added C48: 100n, easypretty:C0603, symbol vesc4-legacy:C-RESCUE-BLDC_4_50
- added C50: 2.2u, easypretty:C0603, symbol vesc4-legacy:C-RESCUE-BLDC_4_48
- added C53: 220n, easypretty:C0603, symbol vesc4-legacy:C-RESCUE-BLDC_4_35
- added H10, H11: Header-Male-2.54_1x2, easypretty:HDR-TH_2P-P2.54-V-M-1, symbol easylib:Header-Male-2.54_1x2
- added L2: BLM18AG601SN1D, easypretty:L0603, symbol easylib:BLM18AG601SN1D
- added R15, R16: 39k, easypretty:R0603, symbol vesc4-legacy:R-RESCUE-BLDC_4_13
- renumbered P3 to ADC/PWR1, P101 to CAN1, P1 to HALL/TEMP1
Connections:
- net +5V: now also ADCbp1.1 (P1), H11.1
- net GND: now also ADCbp1.3 (P3), C48.2, C50.2, C53.2, H10.2, H11.2, R16.1
- net MISO_RX_SCL: now also ADCbp1.7 (P7)
- net RX_SCL_MOSI: now also ADCbp1.6 (P6)
- net TX_SDA: now also ADCbp1.5 (P5)
- net VCC: now also ADCbp1.2 (P2), H10.1, L2.1
- net SCK_ADC_EXT renamed ADC1
- net ADC1: now also R15.1
- new net ADC1_f: ADCbp1.4 (P4), C48.1, R15.2, R16.2
- new net VDDA: C50.1, C53.1, L2.2
