File: Hardware/vesc4-raw/after-remap/mosfets.kicad_sch (KiCad schematic)
At the start: 15 parts, among them Q1 IPT007N06NATMA1, Q2 IPT007N06NATMA1, Q3 IPT007N06NATMA1, Q4 IPT007N06NATMA1, Q5 IPT007N06NATMA1, Q6 IPT007N06NATMA1

Commit message: phase 3 kepasang
mau perbaikin track
Connections:
- net H2_LOW: no longer Q6.2, Q6.3, Q6.4, Q6.5, Q6.6, Q6.7, Q6.8
- net H3_LOW: now also Q6.2, Q6.3, Q6.4, Q6.5, Q6.6, Q6.7, Q6.8
Changed lines of the file:
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@@
+		)
+	)
+	(label "Q4-s"
+		(at 173.99 167.64 0)
+		(effects
+			(font
+				(size 1.27 1.27)
+			)
+			(justify left bottom)
 		)
 	)
@@
 		)
 	)
-	(label "Q4-s"
-		(at 173.99 167.64 0)
-		(effects
-			(font
-				(size 1.27 1.27)
-			)
-			(justify left bottom)
-		)
-	)
 	(label "Q2-g"
 		(at 104.14 143.51 180)
@@
 		)
 	)
-	(label "Q4-s"
+	(label "Q6-s"
 		(at 219.71 167.64 0)
 		(effects
