File: Hardware/vesc4-raw/after-remap/CAN.kicad_sch (KiCad schematic)
At the start: 4 parts, among them U401 SN65HVD232

Commit message: export footprint & ngapus warning unmatched
Parts:
- C401: symbol after-remap-rescue:C-RESCUE-BLDC_4 -> vesc4-legacy:C-RESCUE-BLDC_4_2
- R401: symbol after-remap-rescue:R-RESCUE-BLDC_4 -> vesc4-legacy:R-RESCUE-BLDC_4_3
- R402: symbol after-remap-rescue:R-RESCUE-BLDC_4 -> vesc4-legacy:R-RESCUE-BLDC_4_4
- U401: symbol after-remap-rescue:MCP2551-I/SN-RESCUE-BLDC_4 -> vesc4-legacy:MCP2551-I/SN-RESCUE-BLDC_4_2
Changed lines of the file:
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@@
 	(symbol
 		(lib_name "MCP2551-I/SN-RESCUE-BLDC_4_2")
-		(lib_id "after-remap-rescue:MCP2551-I/SN-RESCUE-BLDC_4")
+		(lib_id "vesc4-legacy:MCP2551-I/SN-RESCUE-BLDC_4_2")
 		(at 148.59 102.87 0)
 		(mirror y)
@@
 	(symbol
 		(lib_name "GND-RESCUE-BLDC_4_6")
-		(lib_id "after-remap-rescue:GND-RESCUE-BLDC_4")
+		(lib_id "vesc4-legacy:GND-RESCUE-BLDC_4_6")
 		(at 148.59 113.03 0)
 		(unit 1)
@@
 	(symbol
 		(lib_name "VCC_3")
-		(lib_id "after-remap-rescue:VCC")
+		(lib_id "vesc4-legacy:VCC_3")
 		(at 148.59 92.71 0)
 		(unit 1)
@@
 	(symbol
 		(lib_name "C-RESCUE-BLDC_4_2")
-		(lib_id "after-remap-rescue:C-RESCUE-BLDC_4")
+		(lib_id "vesc4-legacy:C-RESCUE-BLDC_4_2")
 		(at 156.21 86.36 0)
 		(unit 1)
@@
 	(symbol
 		(lib_name "VCC_4")
-		(lib_id "after-remap-rescue:VCC")
+		(lib_id "vesc4-legacy:VCC_4")
 		(at 156.21 81.28 0)
 		(unit 1)
@@
 	(symbol
 		(lib_name "GND-RESCUE-BLDC_4_5")
-		(lib_id "after-remap-rescue:GND-RESCUE-BLDC_4")
+		(lib_id "vesc4-legacy:GND-RESCUE-BLDC_4_5")
 		(at 156.21 91.44 0)
 		(unit 1)
@@
 	(symbol
 		(lib_name "R-RESCUE-BLDC_4_3")
-		(lib_id "after-remap-rescue:R-RESCUE-BLDC_4")
+		(lib_id "vesc4-legacy:R-RESCUE-BLDC_4_3")
 		(at 124.46 102.87 0)
 		(unit 1)
@@
 	(symbol
 		(lib_name "R-RESCUE-BLDC_4_4")
-		(lib_id "after-remap-rescue:R-RESCUE-BLDC_4")
+		(lib_id "vesc4-legacy:R-RESCUE-BLDC_4_4")
 		(at 162.56 116.84 0)
 		(unit 1)
@@
 	(symbol
 		(lib_name "GND-RESCUE-BLDC_4_4")
-		(lib_id "after-remap-rescue:GND-RESCUE-BLDC_4")
+		(lib_id "vesc4-legacy:GND-RESCUE-BLDC_4_4")
 		(at 162.56 123.19 0)
 		(unit 1)

Commit message: changed footprint 4n7 cap
Parts:
- R402: footprint CRF1:SMD-0603_r -> Library:R0603
Changed lines of the file:
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@@
 			)
 		)
-		(property "Footprint" "CRF1:SMD-0603_r"
+		(property "Footprint" "Library:R0603"
 			(at 160.782 116.84 90)
 			(effects
