File: Hardware/vesc4-raw/after-remap/CAN.kicad_sch (KiCad schematic)
At the start: 4 parts, among them U401 SN65HVD232

Commit message: all done
Parts:
- U401: footprint Library:SOIC-8_L5.0-W4.0-P1.27-LS6.0-BL -> CRF1:SOIC-8-W
Changed lines of the file:
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@@
 			)
 		)
-		(property "Footprint" "Library:SOIC-8_L5.0-W4.0-P1.27-LS6.0-BL"
+		(property "Footprint" "CRF1:SOIC-8-W"
 			(at 148.59 102.87 0)
 			(effects

Commit message: chekcpoint 18 mei
Parts:
- C401: footprint Library:C0603 -> easypretty:C0603; LCSC (none) -> C23630; LCSC Part (none) -> C1631
- R401: footprint Library:R0603 -> easypretty:R0603; LCSC Part (none) -> C23164
- R402: footprint Library:R0603 -> easypretty:R0603; LCSC (none) -> C25804; LCSC Part (none) -> C23164
- U401: LCSC (none) -> C46596301
Changed lines of the file:
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@@
+			)
+		)
+		(property "LCSC" "C46596301"
+			(at 148.59 102.87 0)
+			(effects
+				(font
+					(size 1.27 1.27)
+				)
+				(hide yes)
 			)
 		)
@@
 			)
 		)
-		(property "Footprint" "Library:C0603"
+		(property "Footprint" "easypretty:C0603"
 			(at 157.1752 90.17 0)
 			(effects
@@
 					(size 1.27 1.27)
 				)
+			)
+		)
+		(property "LCSC" "C23630"
+			(at 156.21 86.36 0)
+			(effects
+				(font
+					(size 1.27 1.27)
+				)
+				(hide yes)
+			)
+		)
+		(property "LCSC Part" "C1631"
+			(at 156.21 86.36 0)
+			(effects
+				(font
+					(size 1.27 1.27)
+				)
+				(hide yes)
 			)
 		)
@@
 			)
 		)
-		(property "Footprint" "Library:R0603"
+		(property "Footprint" "easypretty:R0603"
 			(at 122.682 102.87 90)
 			(effects
@@
 		)
 		(property "JLC_3D_Size" "0.81 1.62"
+			(at 124.46 102.87 0)
+			(effects
+				(font
+					(size 1.27 1.27)
+				)
+				(hide yes)
+			)
+		)
+		(property "LCSC Part" "C23164"
 			(at 124.46 102.87 0)
 			(effects
@@
 			)
 		)
-		(property "Footprint" "Library:R0603"
+		(property "Footprint" "easypretty:R0603"
 			(at 160.782 116.84 90)
 			(effects
@@
 			)
 		)
+		(property "LCSC" "C25804"
+			(at 162.56 116.84 0)
+			(effects
+				(font
+					(size 1.27 1.27)
+				)
+				(hide yes)
+			)
+		)
+		(property "LCSC Part" "C23164"
+			(at 162.56 116.84 0)
+			(effects
+				(font
+					(size 1.27 1.27)
+				)
+				(hide yes)
+			)
+		)
