File: Hardware/vesc4-raw/after-remap/Power.kicad_sch (KiCad schematic)
At the start: 48 parts, among them U2 TC2117, U3 DRV8302

Commit message: all done
Parts:
- U2: Manufacturer MICROCHIP(美国微芯) -> (none); Manufacturer Part TC2117-3.3VDBTR -> (none); Supplier LCSC -> (none); Supplier Part C98655 -> (none)
Changed lines of the file:
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@@
-			)
-		)
-		(property "Manufacturer Part" "TC2117-3.3VDBTR"
-			(at 160.02 29.21 0)
-			(effects
-				(font
-					(size 1.27 1.27)
-				)
-				(hide yes)
-			)
-		)
-		(property "Manufacturer" "MICROCHIP(美国微芯)"
-			(at 160.02 29.21 0)
-			(effects
-				(font
-					(size 1.27 1.27)
-				)
-				(hide yes)
-			)
-		)
-		(property "Supplier Part" "C98655"
-			(at 160.02 29.21 0)
-			(effects
-				(font
-					(size 1.27 1.27)
-				)
-				(hide yes)
-			)
-		)
-		(property "Supplier" "LCSC"
-			(at 160.02 29.21 0)
-			(effects
-				(font
-					(size 1.27 1.27)
-				)
-				(hide yes)
 			)
 		)

Commit message: chekcpoint 18 mei
Parts:
- C1, C39, C8: footprint CRF1:SMD-1206 -> easypretty:C1206; JLC_3DModel (none) -> ac9b32e974bc448eab36b1293f859dcb; JLC_3D_Size (none) -> 1.6 0.8; LCSC (none) -> C13585; LCSC Part (none) -> C13585
- C18, C20, C23, C24, C26, C52: footprint Library:C0603 -> easypretty:C0603; LCSC (none) -> C23630; LCSC Part (none) -> C1631
- C19: footprint Library:C0603 -> easypretty:C0603; LCSC (none) -> C107035; LCSC Part (none) -> C1631
- C21: footprint Library:C0603 -> easypretty:C0603; LCSC (none) -> C1631; LCSC Part (none) -> C1631
- C22: footprint Library:C0603 -> easypretty:C0603; LCSC (none) -> C21122; LCSC Part (none) -> C1631
- C25, C33: footprint Library:CAP-SMD_L3.5-W2.8-R-RD -> easypretty:CAP-SMD_L3.5-W2.8-R-RD; LCSC (none) -> C2976906; LCSC Part (none) -> C2976906
- C27: footprint Library:C0603 -> easypretty:C0603; LCSC (none) -> C14663; LCSC Part (none) -> C1631
- C28, C29, C30: footprint Library:C0603 -> easypretty:C0603; LCSC (none) -> C21120; LCSC Part (none) -> C1631
- C34, C36: LCSC (none) -> C1604
- C37: footprint Library:C2220_L5.6-W5.0-H3.0 -> easypretty:C2220; LCSC (none) -> C361175; LCSC Part (none) -> C361175
- C40, C43, C44, C49, C9: footprint Library:C1206 -> easypretty:C1206; LCSC (none) -> C13585; LCSC Part (none) -> C13585
- C51: value 15u, 100v -> 15u,100V; footprint Library:C2220_L5.6-W5.0-H3.0 -> easypretty:C2220; LCSC (none) -> C361175; LCSC Part (none) -> C361175
- D4: JLC_3DModel_Q (none) -> cdc13862fe374d3bb7a14a8cac9d9007; JLC_3D_Size (none) -> 5.05 2.6; LCSC (none) -> C14238
- D5: footprint Library:SOD-123_L2.8-W1.8-LS3.7-RD -> easypretty:SOD-123_L2.8-W1.8-LS3.7-RD; LCSC (none) -> C478011; LCSC Part (none) -> C478011
- L1: footprint Library:IND-SMD_L6.0-W6.0-shield -> easypretty:IND-SMD_L6.0-W6.0; LCSC (none) -> C168080; LCSC Part (none) -> C168080
- R17: footprint Library:R0603 -> easypretty:R0603; LCSC (none) -> C25810; LCSC Part (none) -> C23164
- R18: footprint Library:R0603 -> easypretty:R0603; LCSC (none) -> C22978; LCSC Part (none) -> C23164
- R19: footprint Library:R0603 -> easypretty:R0603; LCSC (none) -> C22809; LCSC Part (none) -> C23164
- R20: footprint Library:R0603 -> easypretty:R0603; LCSC (none) -> C25804; LCSC Part (none) -> C23164
- R21: footprint Library:R0603 -> easypretty:R0603; LCSC (none) -> C22961; LCSC Part (none) -> C23164
- R23, R26, R32: footprint Library:R0603 -> easypretty:R0603; LCSC (none) -> C23153; LCSC Part (none) -> C23164
- R24, R27, R33: footprint Library:R0603 -> easypretty:R0603; LCSC (none) -> C4190; LCSC Part (none) -> C23164
- R25: footprint Library:R0603 -> easypretty:R0603; LCSC (none) -> C22935; LCSC Part (none) -> C23164
- R48, R49, R50, R51: footprint Library:R0603 -> easypretty:R0603; LCSC (none) -> C22775; LCSC Part (none) -> C23164
- U2: footprint Library:SOT-223_L6.5-W3.5-P2.30-LS7.0-BR -> easypretty:SOT-223_L6.5-W3.5-P2.30-LS7.0-BR; LCSC (none) -> C98655; LCSC Part (none) -> C98655
- U3: LCSC (none) -> C84672

Commit message: cp1
Parts:
- added C42, C45, C46: 680u, easypretty:CAP-TH_BD18.0-P7.50-D1.2-FD, symbol Device:C_Polarized
- C1, C40, C43, C44, C49, C8, C9: value 10u,50V -> 10u,100V
- D4: footprint EasyEDA_Lib:SMA_L4.2-W2.6-LS5.1-RD -> easypretty:SOD-123_L2.8-W1.8-LS3.7-RD; LCSC C14238 -> C98663; LCSC Part (none) -> C98663
Connections:
- net GND: now also C42.2, C45.2, C46.2
- net V_SUPPLY: now also C42.1, C45.1, C46.1

Commit message: cp23mei
Parts:
- C1, C40, C43, C44, C49, C8, C9: footprint easypretty:C1206 -> easypretty:C1210; LCSC Part C13585 -> C49326812
- C39: value 10u,50V -> 10u,100V; footprint easypretty:C1206 -> easypretty:C1210; LCSC Part C13585 -> C49326812

Commit message: cp29mei
Connections:
- net S2+: now reaches C36.2, R51.2, U3.30 (SP2)
- net S2-: now reaches C36.1, R50.2, U3.31 (SN2)
- net S1+: now reaches C34.2, R49.2, U3.32 (SP1)
- net S1-: now reaches C34.1, R48.2, U3.33 (SN1)
Changed lines of the file:
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@@
 	(wire
 		(pts
+			(xy 162.56 138.43) (xy 176.53 138.43)
+		)
+		(stroke
+			(width 0)
+			(type default)
+		)
+	)
+	(wire
+		(pts
 			(xy 251.46 97.79) (xy 252.73 97.79)
 		)
@@
 	(wire
 		(pts
-			(xy 176.53 138.43) (xy 162.56 138.43)
-		)
-		(stroke
-			(width 0)
-			(type default)
-		)
-	)
-	(wire
-		(pts
 			(xy 251.46 97.79) (xy 251.46 100.33)
 		)
@@
 		)
 	)
+	(label "S1+"
+		(at 170.18 129.54 0)
+		(effects
+			(font
+				(size 1.27 1.27)
+			)
+			(justify left bottom)
+		)
+	)
+	(label "S2-"
+		(at 166.37 130.81 0)
+		(effects
+			(font
+				(size 1.27 1.27)
+			)
+			(justify left bottom)
+		)
+	)
+	(label "S1-"
+		(at 170.18 121.92 0)
+		(effects
+			(font
+				(size 1.27 1.27)
+			)
+			(justify left bottom)
+		)
+	)
+	(label "S2+"
+		(at 168.91 138.43 0)
+		(effects
+			(font
+				(size 1.27 1.27)
+			)
+			(justify left bottom)
+		)
+	)

Commit message: 16-06-2026
Connections:
- net VCC: no longer U3.24 (REF)
- new net VDDA: U3.24 (REF)
Changed lines of the file:
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@@
 	(wire
 		(pts
-			(xy 96.52 132.08) (xy 96.52 128.27)
-		)
-		(stroke
-			(width 0)
-			(type default)
-		)
-	)
-	(wire
-		(pts
 			(xy 177.8 128.27) (xy 175.26 128.27)
 		)
@@
 		)
 	)
+	(global_label "VDDA"
+		(shape input)
+		(at 96.52 132.08 270)
+		(fields_autoplaced yes)
+		(effects
+			(font
+				(size 1.27 1.27)
+			)
+			(justify right)
+		)
+		(property "Intersheetrefs" "${INTERSHEET_REFS}"
+			(at 96.52 139.1282 90)
+			(effects
+				(font
+					(size 1.27 1.27)
+				)
+				(justify right)
+				(hide yes)
+			)
+		)
+	)
 	(global_label "V_SUPPLY"
 		(shape input)
@@
 					(unit 1)
 				)
-			)
-		)
-	)
-	(symbol
-		(lib_name "VCC_6")
-		(lib_id "vesc4-legacy:VCC_6")
-		(at 96.52 128.27 0)
-		(unit 1)
-		(exclude_from_sim no)
-		(in_bom yes)
-		(on_board yes)
-		(dnp no)
-		(property "Reference" "#PWR062"
-			(at 96.52 125.73 0)
-			(effects
-				(font
-					(size 0.762 0.762)
-				)
-				(hide yes)
-			)
-		)
-		(property "Value" "VCC"
-			(at 96.52 125.73 0)
-			(effects
-				(font
-					(size 0.762 0.762)
-				)
-			)
-		)
-		(property "Footprint" ""
-			(at 96.52 128.27 0)
-			(effects
-				(font
-					(size 1.524 1.524)
-				)
-				(hide yes)
-			)
-		)
-		(property "Datasheet" ""
-			(at 96.52 128.27 0)
-			(effects
-				(font
-					(size 1.524 1.524)
-				)
-				(hide yes)
-			)
-		)
-		(property "Description" ""
-			(at 96.52 128.27 0)
-			(effects
-				(font
-					(size 1.27 1.27)
-				)
-			)
-		)
-		(pin "1"
-		)
-		(instances
-			(project "after-remap"
-				(path "/97cdaedc-7981-4798-95b0-56b9c66aae09/00000000-0000-0000-0000-0000504f83be"
-					(reference "#PWR062")
-					(unit 1)
-				)
