File: Hardware/vesc4-raw/after-remap/hall_filters.kicad_sch (KiCad schematic)
At the start: 11 parts

Commit message: export footprint & ngapus warning unmatched
Parts:
- C4: symbol after-remap-rescue:C-RESCUE-BLDC_4 -> vesc4-legacy:C-RESCUE-BLDC_4_5
- C5: symbol after-remap-rescue:C-RESCUE-BLDC_4 -> vesc4-legacy:C-RESCUE-BLDC_4_6
- C6: symbol after-remap-rescue:C-RESCUE-BLDC_4 -> vesc4-legacy:C-RESCUE-BLDC_4_7
- C7: symbol after-remap-rescue:C-RESCUE-BLDC_4 -> vesc4-legacy:C-RESCUE-BLDC_4_8
- R10: symbol after-remap-rescue:R-RESCUE-BLDC_4 -> vesc4-legacy:R-RESCUE-BLDC_4_10
- R11: symbol after-remap-rescue:R-RESCUE-BLDC_4 -> vesc4-legacy:R-RESCUE-BLDC_4_14
- R12: symbol after-remap-rescue:R-RESCUE-BLDC_4 -> vesc4-legacy:R-RESCUE-BLDC_4_11
- R13: symbol after-remap-rescue:R-RESCUE-BLDC_4 -> vesc4-legacy:R-RESCUE-BLDC_4_12
- R7: symbol after-remap-rescue:R-RESCUE-BLDC_4 -> vesc4-legacy:R-RESCUE-BLDC_4_13
- R8: symbol after-remap-rescue:R-RESCUE-BLDC_4 -> vesc4-legacy:R-RESCUE-BLDC_4_8
- R9: symbol after-remap-rescue:R-RESCUE-BLDC_4 -> vesc4-legacy:R-RESCUE-BLDC_4_9
Changed lines of the file:
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@@
 	(symbol
 		(lib_name "R-RESCUE-BLDC_4_13")
-		(lib_id "after-remap-rescue:R-RESCUE-BLDC_4")
+		(lib_id "vesc4-legacy:R-RESCUE-BLDC_4_13")
 		(at 124.46 81.28 180)
 		(unit 1)
@@
 	(symbol
 		(lib_name "R-RESCUE-BLDC_4_8")
-		(lib_id "after-remap-rescue:R-RESCUE-BLDC_4")
+		(lib_id "vesc4-legacy:R-RESCUE-BLDC_4_8")
 		(at 140.97 95.25 90)
 		(unit 1)
@@
 	(symbol
 		(lib_name "R-RESCUE-BLDC_4_9")
-		(lib_id "after-remap-rescue:R-RESCUE-BLDC_4")
+		(lib_id "vesc4-legacy:R-RESCUE-BLDC_4_9")
 		(at 140.97 92.71 90)
 		(unit 1)
@@
 	(symbol
 		(lib_name "R-RESCUE-BLDC_4_10")
-		(lib_id "after-remap-rescue:R-RESCUE-BLDC_4")
+		(lib_id "vesc4-legacy:R-RESCUE-BLDC_4_10")
 		(at 140.97 90.17 90)
 		(unit 1)
@@
 	(symbol
 		(lib_name "C-RESCUE-BLDC_4_6")
-		(lib_id "after-remap-rescue:C-RESCUE-BLDC_4")
+		(lib_id "vesc4-legacy:C-RESCUE-BLDC_4_6")
 		(at 151.13 107.95 0)
 		(unit 1)
@@
 	(symbol
 		(lib_name "C-RESCUE-BLDC_4_7")
-		(lib_id "after-remap-rescue:C-RESCUE-BLDC_4")
+		(lib_id "vesc4-legacy:C-RESCUE-BLDC_4_7")
 		(at 157.48 107.95 0)
 		(unit 1)
@@
 	(symbol
 		(lib_name "C-RESCUE-BLDC_4_8")
-		(lib_id "after-remap-rescue:C-RESCUE-BLDC_4")
+		(lib_id "vesc4-legacy:C-RESCUE-BLDC_4_8")
 		(at 163.83 107.95 0)
 		(unit 1)
@@
 	(symbol
 		(lib_name "GND-RESCUE-BLDC_4_6")
-		(lib_id "after-remap-rescue:GND-RESCUE-BLDC_4")
+		(lib_id "vesc4-legacy:GND-RESCUE-BLDC_4_6")
 		(at 151.13 113.03 0)
 		(unit 1)
@@
 	(symbol
 		(lib_name "R-RESCUE-BLDC_4_14")
-		(lib_id "after-remap-rescue:R-RESCUE-BLDC_4")
+		(lib_id "vesc4-legacy:R-RESCUE-BLDC_4_14")
 		(at 127 81.28 180)
 		(unit 1)
@@
 	(symbol
 		(lib_name "R-RESCUE-BLDC_4_11")
-		(lib_id "after-remap-rescue:R-RESCUE-BLDC_4")
+		(lib_id "vesc4-legacy:R-RESCUE-BLDC_4_11")
 		(at 129.54 81.28 180)
 		(unit 1)
@@
 	(symbol
 		(lib_name "R-RESCUE-BLDC_4_12")
-		(lib_id "after-remap-rescue:R-RESCUE-BLDC_4")
+		(lib_id "vesc4-legacy:R-RESCUE-BLDC_4_12")
 		(at 132.08 81.28 180)
 		(unit 1)
@@
 	(symbol
 		(lib_name "C-RESCUE-BLDC_4_5")
-		(lib_id "after-remap-rescue:C-RESCUE-BLDC_4")
+		(lib_id "vesc4-legacy:C-RESCUE-BLDC_4_5")
 		(at 129.54 107.95 180)
 		(unit 1)
@@
 	(symbol
 		(lib_name "GND-RESCUE-BLDC_4_5")
-		(lib_id "after-remap-rescue:GND-RESCUE-BLDC_4")
+		(lib_id "vesc4-legacy:GND-RESCUE-BLDC_4_5")
 		(at 129.54 113.03 0)
 		(unit 1)
@@
 	(symbol
 		(lib_name "VCC_2")
-		(lib_id "after-remap-rescue:VCC")
+		(lib_id "vesc4-legacy:VCC_2")
 		(at 124.46 72.39 0)
 		(unit 1)
@@
 	(symbol
 		(lib_name "GND-RESCUE-BLDC_4_7")
-		(lib_id "after-remap-rescue:GND-RESCUE-BLDC_4")
+		(lib_id "vesc4-legacy:GND-RESCUE-BLDC_4_7")
 		(at 157.48 113.03 0)
 		(unit 1)
@@
 	(symbol
 		(lib_name "GND-RESCUE-BLDC_4_8")
-		(lib_id "after-remap-rescue:GND-RESCUE-BLDC_4")
+		(lib_id "vesc4-legacy:GND-RESCUE-BLDC_4_8")
 		(at 163.83 113.03 0)
 		(unit 1)

Commit message: cp sebelum ganti 4n7
Parts:
- C4, C5, C6, C7: footprint CRF1:SMD-0603_c -> Library:C0603
Changed lines of the file:
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@@
 			)
 		)
-		(property "Footprint" "CRF1:SMD-0603_c"
+		(property "Footprint" "Library:C0603"
 			(at 151.13 107.95 0)
 			(effects
@@
 			)
 		)
-		(property "Footprint" "CRF1:SMD-0603_c"
+		(property "Footprint" "Library:C0603"
 			(at 157.48 107.95 0)
 			(effects
@@
 			)
 		)
-		(property "Footprint" "CRF1:SMD-0603_c"
+		(property "Footprint" "Library:C0603"
 			(at 163.83 107.95 0)
 			(effects
@@
 			)
 		)
-		(property "Footprint" "CRF1:SMD-0603_c"
+		(property "Footprint" "Library:C0603"
 			(at 129.54 107.95 0)
 			(effects

Commit message: changed footprint 4n7 cap
Parts:
- R12: footprint CRF1:SMD-0603_r -> Library:R0603
Changed lines of the file:
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@@
 			)
 		)
-		(property "Footprint" "CRF1:SMD-0603_r"
+		(property "Footprint" "Library:R0603"
 			(at 129.54 81.28 0)
 			(effects
