File: Hardware/vesc4-raw/after-remap/STM32F4 64LQFP.kicad_sch (KiCad schematic)
At the start: 15 parts, among them P2 SWD, U1 STM32F40X_LQFP64, X2 5TJ480000NYLBC

Commit message: all done
Parts:
- P2: footprint CRF1:MICRO_JST_6 -> Library:CONN-TH_B6B-PH-K-S
Changed lines of the file:
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@@
 			)
 		)
-		(property "Footprint" "CRF1:MICRO_JST_6"
+		(property "Footprint" "Library:CONN-TH_B6B-PH-K-S"
 			(at 256.54 80.01 0)
 			(effects

Commit message: chekcpoint 18 mei
Parts:
- C10, C11, C12, C13, C14, C16, C17, C31, C35: footprint Library:C0603 -> easypretty:C0603; LCSC (none) -> C23630; LCSC Part (none) -> C1631
- C15, C38: footprint Library:C0603 -> easypretty:C0603; LCSC (none) -> C1644; LCSC Part (none) -> C1631
- C32: footprint Library:C0603 -> easypretty:C0603; LCSC (none) -> C14663; LCSC Part (none) -> C1631
- P2: footprint Library:CONN-TH_B6B-PH-K-S -> easypretty:CONN-TH_B6B-PH-K-S
- U1: LCSC (none) -> C15742
- X2: footprint Library:C2149245 -> easypretty:CRYSTAL-SMD_4P-L5.0-W3.2-BL; LCSC (none) -> C2149245; LCSC Part (none) -> C2149245

Commit message: 16-06-2026
Parts:
- renumbered P2 to SWD1
Connections:
- net VCC: no longer C31.2, U1.13 (VDDA)
- new net VDDA: C31.2, U1.13 (VDDA)
Other:
- moved on the sheet: C31
Changed lines of the file:
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@@
 	)
 	(junction
+		(at 190.5 146.05)
+		(diameter 0)
+		(color 0 0 0 0)
+	)
+	(junction
 		(at 196.85 146.05)
 		(diameter 0)
@@
 	)
 	(junction
-		(at 196.85 130.81)
+		(at 187.96 133.35)
 		(diameter 0)
 		(color 0 0 0 0)
@@
 	)
 	(junction
-		(at 187.96 130.81)
-		(diameter 0)
-		(color 0 0 0 0)
-	)
-	(junction
 		(at 182.88 128.27)
 		(diameter 0)
@@
 	(wire
 		(pts
-			(xy 187.96 130.81) (xy 187.96 143.51)
-		)
-		(stroke
-			(width 0)
-			(type default)
-		)
-	)
-	(wire
-		(pts
 			(xy 203.2 146.05) (xy 203.2 153.67)
 		)
@@
 	(wire
 		(pts
+			(xy 190.5 146.05) (xy 196.85 146.05)
+		)
+		(stroke
+			(width 0)
+			(type default)
+		)
+	)
+	(wire
+		(pts
 			(xy 196.85 161.29) (xy 195.58 161.29)
 		)
@@
 	(wire
 		(pts
-			(xy 196.85 143.51) (xy 196.85 146.05)
+			(xy 251.46 25.4) (xy 251.46 27.94)
 		)
 		(stroke
@@
 	(wire
 		(pts
-			(xy 251.46 25.4) (xy 251.46 27.94)
+			(xy 228.6 52.07) (xy 231.14 52.07)
 		)
 		(stroke
@@
 		)
 	)
-	(wire
+	(polyline
 		(pts
-			(xy 187.96 129.54) (xy 187.96 130.81)
+			(xy 234.95 67.31) (xy 234.95 90.17)
 		)
 		(stroke
 			(width 0)
-			(type default)
+			(type dash)
 		)
 	)
 	(wire
 		(pts
-			(xy 228.6 52.07) (xy 231.14 52.07)
+			(xy 187.96 130.81) (xy 187.96 133.35)
 		)
 		(stroke
@@
 		)
 	)
-	(polyline
-		(pts
-			(xy 234.95 67.31) (xy 234.95 90.17)
-		)
-		(stroke
-			(width 0)
-			(type dash)
-		)
-	)
 	(wire
 		(pts
@@
 		)
 	)
-	(wire
-		(pts
-			(xy 196.85 133.35) (xy 196.85 130.81)
-		)
-		(stroke
-			(width 0)
-			(type default)
-		)
-	)
 	(polyline
 		(pts
@@
 	(wire
 		(pts
-			(xy 177.8 146.05) (xy 196.85 146.05)
+			(xy 177.8 146.05) (xy 190.5 146.05)
+		)
+		(stroke
+			(width 0)
+			(type default)
+		)
+	)
+	(wire
+		(pts
+			(xy 187.96 143.51) (xy 187.96 133.35)
 		)
 		(stroke
@@
 	(wire
 		(pts
-			(xy 187.96 130.81) (xy 196.85 130.81)
+			(xy 190.5 143.51) (xy 190.5 146.05)
 		)
 		(stroke
@@
 	(wire
 		(pts
+			(xy 187.96 133.35) (xy 190.5 133.35)
+		)
+		(stroke
+			(width 0)
+			(type default)
+		)
+	)
+	(wire
+		(pts
 			(xy 245.11 69.85) (xy 245.11 73.66)
 		)
@@
 		)
 	)
+	(global_label "VDDA"
+		(shape input)
+		(at 187.96 130.81 90)
+		(fields_autoplaced yes)
+		(effects
+			(font
+				(size 1.27 1.27)
+			)
+			(justify left)
+		)
+		(property "Intersheetrefs" "${INTERSHEET_REFS}"
+			(at 187.96 123.7618 90)
+			(effects
+				(font
+					(size 1.27 1.27)
+				)
+				(justify left)
+				(hide yes)
+			)
+		)
+	)
 	(hierarchical_label "SENS3"
 		(shape input)
@@
 		(lib_name "VCC_9")
 		(lib_id "vesc4-legacy:VCC_9")
-		(at 187.96 129.54 0)
+		(at 196.85 130.81 0)
 		(unit 1)
 		(exclude_from_sim no)
@@
 		(dnp no)
 		(property "Reference" "#PWR036"
-			(at 187.96 127 0)
+			(at 196.85 128.27 0)
 			(effects
 				(font
@@
 		)
 		(property "Value" "VCC"
-			(at 187.96 127 0)
+			(at 196.85 128.27 0)
 			(effects
 				(font
@@
 		)
 		(property "Footprint" ""
-			(at 187.96 129.54 0)
+			(at 196.85 130.81 0)
 			(effects
 				(font
@@
 		)
 		(property "Datasheet" ""
-			(at 187.96 129.54 0)
+			(at 196.85 130.81 0)
 			(effects
 				(font
@@
 		)
 		(property "Description" ""
-			(at 187.96 129.54 0)
+			(at 196.85 130.81 0)
 			(effects
 				(font
@@
 		(lib_name "C-RESCUE-BLDC_4_22")
 		(lib_id "vesc4-legacy:C-RESCUE-BLDC_4_22")
-		(at 196.85 138.43 180)
+		(at 190.5 138.43 180)
 		(unit 1)
 		(exclude_from_sim no)
@@
 		(dnp no)
 		(property "Reference" "C31"
-			(at 195.58 140.97 0)
+			(at 189.23 140.97 0)
 			(effects
 				(font
@@
 		)
 		(property "Value" "2.2u"
-			(at 195.58 135.89 0)
+			(at 189.23 135.89 0)
 			(effects
 				(font
@@
 		)
 		(property "Footprint" "easypretty:C0603"
-			(at 196.85 138.43 0)
+			(at 190.5 138.43 0)
 			(effects
 				(font
@@
 		)
 		(property "Datasheet" ""
-			(at 196.85 138.43 0)
+			(at 190.5 138.43 0)
 			(effects
 				(font
@@
 		)
 		(property "Description" ""
-			(at 196.85 138.43 0)
+			(at 190.5 138.43 0)
 			(effects
 				(font
@@
 		)
 		(property "LCSC" "C23630"
-			(at 196.85 138.43 0)
+			(at 190.5 138.43 0)
 			(effects
 				(font
@@
 		)
 		(property "LCSC Part" "C1631"
-			(at 196.85 138.43 0)
+			(at 190.5 138.43 0)
 			(effects
 				(font
@@
 		)
 		(property "mfg#" ""
-			(at 196.85 138.43 0)
+			(at 190.5 138.43 0)
 			(effects
 				(font
@@
 		(on_board yes)
 		(dnp no)
-		(property "Reference" "P2"
+		(property "Reference" "SWD1"
 			(at 255.27 80.01 90)
 			(effects
@@
 			(project "after-remap"
 				(path "/97cdaedc-7981-4798-95b0-56b9c66aae09/00000000-0000-0000-0000-000053f7501a"
-					(reference "P2")
+					(reference "SWD1")
 					(unit 1)
 				)
